Commit message: readme update

File: hyperspawn/dropbear.urdf (robot description, URDF)
Before this commit: robot humanoid, 666 links, 665 joints
Joints:
- joint head_Revolute_26: limit (none) -> effort=1.0 velocity=10.0
- joint head_Revolute_27: limit (none) -> effort=1.0 velocity=10.0
- joint head_Revolute_34: limit (none) -> effort=1.0 velocity=10.0
- joint head_Revolute_37: limit (none) -> effort=1.0 velocity=10.0
- joint head_Revolute_38: limit (none) -> effort=1.0 velocity=10.0
- joint head_Revolute_44: limit (none) -> effort=1.0 velocity=10.0
- joint head_Revolute_45: limit (none) -> effort=1.0 velocity=10.0
- joint head_Revolute_47: limit (none) -> effort=1.0 velocity=10.0
- joint head_Revolute_48: limit (none) -> effort=1.0 velocity=10.0
- joint head_Revolute_54: limit (none) -> effort=1.0 velocity=10.0
- joint head_Revolute_55: limit (none) -> effort=1.0 velocity=10.0
- joint head_Revolute_57: limit (none) -> effort=1.0 velocity=10.0
- joint head_Revolute_58: limit (none) -> effort=1.0 velocity=10.0
- joint head_Revolute_64: limit (none) -> effort=1.0 velocity=10.0
- joint head_Revolute_65: limit (none) -> effort=1.0 velocity=10.0
- joint head_Revolute_67: limit (none) -> effort=1.0 velocity=10.0
- joint head_Revolute_68: limit (none) -> effort=1.0 velocity=10.0
- joint head_Revolute_74: limit (none) -> effort=1.0 velocity=10.0
- joint head_Revolute_75: limit (none) -> effort=1.0 velocity=10.0
- joint head_Revolute_77: limit (none) -> effort=1.0 velocity=10.0
- joint head_Revolute_78: limit (none) -> effort=1.0 velocity=10.0
- joint head_Revolute_84: limit (none) -> effort=1.0 velocity=10.0
- joint head_Revolute_85: limit (none) -> effort=1.0 velocity=10.0
